Commit message: xacro file

File: src/my_arm_description/urdf/six_dof_arm.urdf (robot description, URDF)
Before this commit: robot six_dof_arm, 7 links, 6 joints
Links:
- removed link link_1
- removed link link_2
- removed link link_3
- removed link link_4
- removed link link_5
- link base_link: mass 1 -> None; geometry collision cylinder length=${base_height} radius=${base_radius}; visual cylinder length=${base_height} radius=${base_radius}
- link tool0: geometry collision box size=0.05 0.05 ${tool_len}; visual box size=0.05 0.05 ${tool_len}
Joints:
- joint joint_1: limit lower=-3.1416 upper=3.1416 effort=10 velocity=1.57 -> lower=-3.14 upper=3.14 effort=10 velocity=1.5; origin xyz=0 0 0.05 rpy=0 0 0 -> xyz=0 0 ${base_height} rpy=0 0 0
- joint joint_2: limit lower=-1.5708 upper=1.5708 effort=10 velocity=1.57 -> lower=-1.57 upper=1.57 effort=10 velocity=1.5; origin xyz=0 0 0.30 rpy=0 0 0 -> xyz=0 0 ${l1_len} rpy=0 0 0
- joint joint_3: limit lower=-1.5708 upper=1.5708 effort=8 velocity=1.57 -> lower=-1.57 upper=1.57 effort=8 velocity=1.5; origin xyz=0 0 0.30 rpy=0 0 0 -> xyz=0 0 ${l2_len} rpy=0 0 0
- joint joint_4: limit lower=-1.5708 upper=1.5708 effort=5 velocity=2.09 -> lower=-1.57 upper=1.57 effort=5 velocity=2.0; origin xyz=0 0 0.30 rpy=0 0 0 -> xyz=0 0 ${l3_len} rpy=0 0 0
- joint joint_5: limit lower=-1.5708 upper=1.5708 effort=4 velocity=2.09 -> lower=-1.57 upper=1.57 effort=4 velocity=2.0; origin xyz=0 0 0.20 rpy=0 0 0 -> xyz=0 0 ${l4_len} rpy=0 0 0
- joint joint_6: limit lower=-3.1416 upper=3.1416 effort=2 velocity=2.09 -> lower=-3.14 upper=3.14 effort=2 velocity=2.0; origin xyz=0 0 0.10 rpy=0 0 0 -> xyz=0 0 ${l5_len} rpy=0 0 0
